Commit message: fix: lower gripper URDF joint limit to -0.030 so overshoot reaches motor

File: src/openarm_description/urdf/ee/openarm_hand.xacro (robot description, xacro)
@@ -60,5 +60,5 @@
       <origin xyz="0 -0.006 0.015" rpy="0 0 0" />
       <axis xyz="0 -1 0" />
-      <limit effort="333" lower="0.0" upper="0.044" velocity="10.0" />
+      <limit effort="333" lower="-0.030" upper="0.044" velocity="10.0" />
     </joint>
     <joint name="${ee_prefix}finger_joint2" type="prismatic">
